File: Mini-3p3V-Supply.kicad_pcb (KiCad board)
At the start: 2 copper layers, 26 x 12 mm, 7 parts, among them J1 5V, J2 Gnd, J3 3.3V, J4 Gnd, J5 USB_OTG, U1 LM1117-3.3

Commit message: It works
Parts:
- J5: footprint Connectors_USB_Local:USB_Micro_B_FCI_10118192 -> Project_Local:USB_Micro_B_FCI_10118192_HandSolder
Connections:
- J5 pad 2: (no net) -> Net-(J5-Pad2)
- J5 pad 3: (no net) -> Net-(J5-Pad3)
- J5 pad 4: (no net) -> Net-(J5-Pad4)
Routing:
- net +5V: track 6.38 -> 5.63 mm, vias 2 -> 1
Other:
- board text added: "3.3V"
- board text added: "Gnd"
- board text added: "Jacob M. 9/21/2018 V0.2.0 5V to 3.3V"
- board text removed: "Jacob M. 9/12/2018 V0.1 5V to 3.3V"
Changed lines of the file:
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@@
     (area 125.434287 101.6 175.17 128.000001)
     (thickness 1.6)
-    (drawings 11)
-    (tracks 41)
+    (drawings 14)
+    (tracks 39)
     (zones 0)
     (modules 7)
-    (nets 4)
+    (nets 7)
   )
   (page A4)
@@
   (net 2 GND)
   (net 3 +5V)
+  (net 4 "Net-(J5-Pad2)")
+  (net 5 "Net-(J5-Pad3)")
+  (net 6 "Net-(J5-Pad4)")
   (net_class Default "This is the default net class."
     (clearance 0.1524)
@@
     (uvia_drill 0.3302)
     (add_net GND)
+    (add_net "Net-(J5-Pad2)")
+    (add_net "Net-(J5-Pad3)")
+    (add_net "Net-(J5-Pad4)")
   )
   (net_class PWR ""
@@
     (add_net +3V3)
     (add_net +5V)
-  )
-  (module Connectors_USB_Local:USB_Micro_B_FCI_10118192 (layer B.Cu)
-    (at 138.52 114.3)
-    (descr https://github.com/JoanTheSpark/KiCAD)
-    (fp_text reference J5 (at 1.4732 0.0635 90) (layer B.SilkS)
-      (effects (font (size 0.7 0.7) (thickness 0.15)) (justify mirror))
-    )
-    (fp_text value USB_OTG (at 5.08 0 270) (layer B.Fab)
-      (effects (font (size 1 1) (thickness 0.15)) (justify mirror))
-    )
-    (fp_line (start 3.6 -3.7) (end -1.45 -3.7) (layer B.CrtYd) (width 0.15))
-    (fp_line (start 3.6 3.7) (end 3.6 -3.7) (layer B.CrtYd) (width 0.15))
-    (fp_line (start -1.45 3.7) (end 3.6 3.7) (layer B.CrtYd) (width 0.15))
-    (fp_line (start -1.45 3.7) (end -1.45 -3.7) (layer B.CrtYd) (width 0.15))
-    (pad 1 smd rect (at 3 1.3) (size 2 0.4) (layers B.Cu B.Paste B.Mask)
-      (net 3 +5V) (solder_mask_margin 0.0762) (solder_paste_margin -0.0762) (clearance 0.0762))
-    (pad 2 smd rect (at 2.8 0.65) (size 1.6 0.4) (layers B.Cu B.Paste B.Mask)
-      (solder_mask_margin 0.0762) (solder_paste_margin -0.0762) (clearance 0.0762))
-    (pad 3 smd rect (at 2.8 0) (size 1.6 0.4) (layers B.Cu B.Paste B.Mask)
-      (solder_mask_margin 0.0762) (solder_paste_margin -0.0762) (clearance 0.0762))
-    (pad 4 smd rect (at 2.8 -0.65) (size 1.6 0.4) (layers B.Cu B.Paste B.Mask)
-      (solder_mask_margin 0.0762) (solder_paste_margin -0.0762) (clearance 0.0762))
-    (pad 5 smd rect (at 2.8 -1.3) (size 1.6 0.4) (layers B.Cu B.Paste B.Mask)
-      (net 2 GND) (solder_mask_margin 0.0762) (solder_paste_margin -0.0762) (clearance 0.0762))
-    (pad 6 smd rect (at 0 3.8) (size 1.9 1.9) (layers B.Cu B.Paste B.Mask)
-      (net 2 GND) (solder_mask_margin 0.0762) (solder_paste_margin -0.0762) (clearance 0.0762))
-    (pad 6 smd rect (at 0 -3.8) (size 1.9 1.9) (layers B.Cu B.Paste B.Mask)
-      (net 2 GND) (solder_mask_margin 0.0762) (solder_paste_margin -0.0762) (clearance 0.0762))
-    (pad 6 smd rect (at 2.55 -3.1) (size 1.6 2.1) (layers B.Cu B.Paste B.Mask)
-      (net 2 GND) (solder_mask_margin 0.0762) (solder_paste_margin -0.0762) (clearance 0.0762))
-    (pad 6 smd rect (at 2.55 3.1) (size 1.6 2.1) (layers B.Cu B.Paste B.Mask)
-      (net 2 GND) (solder_mask_margin 0.0762) (clearance 0.0762))
-    (pad 6 smd rect (at 0 -1.2) (size 1.9 1.9) (layers B.Cu B.Paste B.Mask)
-      (net 2 GND) (solder_mask_margin 0.0762) (solder_paste_margin -0.0762) (clearance 0.0762))
-    (pad 6 smd rect (at 0 1.2) (size 1.9 1.9) (layers B.Cu B.Paste B.Mask)
-      (net 2 GND) (solder_mask_margin 0.0762) (solder_paste_margin -0.0762) (clearance 0.0762))
-    (model Connectors_USB.3dshapes/Conn_USB-micro-2.0_socket_right-angle.wrl
-      (at (xyz 0 0 0))
-      (scale (xyz 1 1 1))
-      (rotate (xyz 0 0 0))
-    )
   )
   (module Capacitors_Tantalum_SMD:CP_Tantalum_Case-C_EIA-6032-28_Hand (layer F.Cu)
@@
       (net 2 GND))
   )
+  (module Project_Local:USB_Micro_B_FCI_10118192_HandSolder (layer B.Cu)
+    (at 138.52 114.3)
+    (descr https://github.com/JoanTheSpark/KiCAD)
+    (fp_text reference J5 (at 1.4732 0.0635 90) (layer B.SilkS)
+      (effects (font (size 0.7 0.7) (thickness 0.15)) (justify mirror))
+    )
+    (fp_text value USB_OTG (at 5.08 0 270) (layer B.Fab)
+      (effects (font (size 1 1) (thickness 0.15)) (justify mirror))
+    )
+    (fp_line (start 3.6 -3.7) (end -1.45 -3.7) (layer B.CrtYd) (width 0.15))
+    (fp_line (start 3.6 3.7) (end 3.6 -3.7) (layer B.CrtYd) (width 0.15))
+    (fp_line (start -1.45 3.7) (end 3.6 3.7) (layer B.CrtYd) (width 0.15))
+    (fp_line (start -1.45 3.7) (end -1.45 -3.7) (layer B.CrtYd) (width 0.15))
+    (pad 1 smd rect (at 3.5 1.3) (size 3 0.4) (layers B.Cu B.Paste B.Mask)
+      (net 3 +5V) (solder_mask_margin 0.0762) (solder_paste_margin -0.0762) (clearance 0.0762))
+    (pad 2 smd rect (at 3.5 0.65) (size 3 0.4) (layers B.Cu B.Paste B.Mask)
+      (net 4 "Net-(J5-Pad2)") (solder_mask_margin 0.0762) (solder_paste_margin -0.0762) (clearance 0.0762))
+    (pad 3 smd rect (at 3.5 0) (size 3 0.4) (layers B.Cu B.Paste B.Mask)
+      (net 5 "Net-(J5-Pad3)") (solder_mask_margin 0.0762) (solder_paste_margin -0.0762) (clearance 0.0762))
+    (pad 4 smd rect (at 3.5 -0.65) (size 3 0.4) (layers B.Cu B.Paste B.Mask)
+      (net 6 "Net-(J5-Pad4)") (solder_mask_margin 0.0762) (solder_paste_margin -0.0762) (clearance 0.0762))
+    (pad 5 smd rect (at 3.5 -1.3) (size 3 0.4) (layers B.Cu B.Paste B.Mask)
+      (net 2 GND) (solder_mask_margin 0.0762) (solder_paste_margin -0.0762) (clearance 0.0762))
+    (pad 6 smd rect (at 0 3.8) (size 1.9 1.9) (layers B.Cu B.Paste B.Mask)
+      (net 2 GND) (solder_mask_margin 0.0762) (solder_paste_margin -0.0762) (clearance 0.0762))
+    (pad 6 smd rect (at 0 -3.8) (size 1.9 1.9) (layers B.Cu B.Paste B.Mask)
+      (net 2 GND) (solder_mask_margin 0.0762) (solder_paste_margin -0.0762) (clearance 0.0762))
+    (pad 6 smd rect (at 2.55 -3.1) (size 1.6 2.1) (layers B.Cu B.Paste B.Mask)
+      (net 2 GND) (solder_mask_margin 0.0762) (solder_paste_margin -0.0762) (clearance 0.0762))
+    (pad 6 smd rect (at 2.55 3.1) (size 1.6 2.1) (layers B.Cu B.Paste B.Mask)
+      (net 2 GND) (solder_mask_margin 0.0762) (clearance 0.0762))
+    (pad 6 smd rect (at 0 -1.2) (size 1.9 1.9) (layers B.Cu B.Paste B.Mask)
+      (net 2 GND) (solder_mask_margin 0.0762) (solder_paste_margin -0.0762) (clearance 0.0762))
+    (pad 6 smd rect (at 0 1.2) (size 1.9 1.9) (layers B.Cu B.Paste B.Mask)
+      (net 2 GND) (solder_mask_margin 0.0762) (solder_paste_margin -0.0762) (clearance 0.0762))
+    (model Connectors_USB.3dshapes/Conn_USB-micro-2.0_socket_right-angle.wrl
+      (at (xyz 0 0 0))
+      (scale (xyz 1 1 1))
+      (rotate (xyz 0 0 0))
+    )
+  )
+  (gr_text OUT (at 160.82 114.3) (layer B.SilkS)
+    (effects (font (size 1 1) (thickness 0.15)) (justify mirror))
+  )
+  (gr_text 3.3V (at 160.82 119.5) (layer B.SilkS)
+    (effects (font (size 1 1) (thickness 0.15)) (justify mirror))
+  )
+  (gr_text Gnd (at 160.82 109.1) (layer B.SilkS)
+    (effects (font (size 1 1) (thickness 0.15)) (justify mirror))
+  )
   (gr_text IN (at 139.82 114.3) (layer F.SilkS)
     (effects (font (size 1 1) (thickness 0.15)))
   )
-  (gr_text "Jacob M.\n9/12/2018\nV0.1\n5V to 3.3V" (at 152.32 114.3) (layer B.SilkS)
+  (gr_text "Jacob M.\n9/21/2018\nV0.2.0\n5V to 3.3V" (at 152.32 114.3) (layer B.SilkS)
     (effects (font (size 1 1) (thickness 0.15)) (justify mirror))
   )
@@
   (segment (start 144.17 112) (end 144.02 112) (width 0.1524) (layer F.Cu) (net 2) (status 30))
   (segment (start 144.02 112) (end 143.32 111.3) (width 0.1524) (layer F.Cu) (net 2) (status 30))
-  (segment (start 144.17 116.6) (end 143.42 116.6) (width 1.27) (layer F.Cu) (net 3))
-  (segment (start 143.42 116.6) (end 142.72 115.9) (width 1.27) (layer F.Cu) (net 3))
-  (via (at 142.72 115.9) (size 0.6858) (drill 0.3302) (layers F.Cu B.Cu) (net 3))
+  (segment (start 139.82 117.3) (end 143.47 117.3) (width 1.27) (layer F.Cu) (net 3))
+  (segment (start 143.47 117.3) (end 144.17 116.6) (width 1.27) (layer F.Cu) (net 3))
   (via (at 144.17 116.6) (size 0.6858) (drill 0.3302) (layers F.Cu B.Cu) (net 3))
-  (segment (start 144.17 116.6) (end 140.52 116.6) (width 1.27) (layer F.Cu) (net 3))
   (segment (start 140.52 116.6) (end 139.82 117.3) (width 1.27) (layer F.Cu) (net 3))
   (zone (net 2) (net_name GND) (layer F.Cu) (hatch edge 0.508)
@@
     (polygon
       (pts
-        (xy 140.52 115.4) (xy 140.52 115.8) (xy 142.02 115.8) (xy 142.92 116.7) (xy 142.92 117.4)
-        (xy 145.22 117.4) (xy 145.22 115.8) (xy 143.12 115.8) (xy 142.72 115.4)
+        (xy 140.52 115.4) (xy 140.52 115.8) (xy 142.62 115.8) (xy 143.12 116.3) (xy 143.12 117.4)
+        (xy 145.22 117.4) (xy 145.22 115.8) (xy 143.92 115.8) (xy 143.52 115.4)
       )
     )
